File: EsquemaKicad/Coche teledirigido-backups/Backup_20253017/Coche teledirigido.kicad_sch (KiCad schematic)
At the start: 66 parts, among them J1 Conn_VCC_1M, J10 Conn_LDR_F, J11 Conn_Servo1_F, J12 Conn_M1_F, J13 Conn_BZ_F, J2 Conn_VCC_2M, J3 Conn_VCC_1H, J4 Conn_VCC_2H, J5 ESP32-C3, J6 Conn_LDR_M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

Commit message: Nueva versión
Parts:
- removed R23, R24: 10kΩ, symbol caca-coche-rescue:R
- R21: value 5kΩ -> 10kΩ
- renumbered R25 to R23, R26 to R24
Connections:
- net SEN5 is gone; now on net LDR5: J5.3 (Pin_3)
- net +5v (2.600mA): no longer U4.4, U5.4
- net at R24.1, U5.1: now also U5.4
- net SEN4: now reaches U5.3
- net SEN4: now also J5.2 (Pin_2)
- net at R23.1, U4.1: now also U4.4
- net SEN3: now reaches U4.3
- net SEN3: now also J5.1 (Pin_1)
- net LDR3 renamed LDR5
- net LDR5: no longer J5.1 (Pin_1)
- net LUZ STOP renamed LUZ MATR
- net SEN2: no longer names the net of J5.14 (Pin_14)
Other:
- note added: "PWM0 PIN0 OUT PWM PWM1 PIN1 OUT PWM SEN3 PIN3 IN ANALOG SEN4 PIN4 IN ANALOG LDR5 PIN5 IN ANALOG PWM6 PIN6 OUT PWM PWM7 PIN7 OUT PWM SER8 PIN8 OUT DIGITAL SRCLK9 PIN9 OUT DIGITAL RCLK10 PIN10 OUT DIGITAL"
- note removed: "PWM0 PIN0 OUT PWM PWM1 PIN1 OUT PWM SEN2 PIN2 IN ANALOG LDR3 PIN3 IN ANALOG SEN5 PIN5 IN ANALOG PWM6 PIN6 OUT PWM PWM7 PIN7 OUT PWM SER8 PIN8 OUT DIGITAL SRCLK9 PIN9 OUT DIGITAL RCLK10 PIN10 OUT DIGITAL"
- title: Esquema Coche Teledirigido 2.2 -> Esquema Coche Teledirigido 2
- moved on the sheet: U5
